File: Ring_Mod_Wave_Folder/Ring_fold_main/Ring_fold_main.sch (KiCad schematic (older format))
At the start: 40 parts, among them IC1 AD633, J1 Conn_Eurorack_5, Q1 2N3904, U1 TL072, U2 TL072, U3 TL072

Commit message: Add panel and gerbers
Parts:
- R1, R10, R11, R12, R13, R14, R15, R16, R17, R18, R19, R2, R20, R21, R22, R3, R4, R5, R6, R7, R8, R9: footprint Resistor_THT:R_Axial_Default -> Resistor_THT:R_Axial_DIN0204_L3.6mm_D1.6mm_P5.08mm_Horizontal
Changed lines of the file:
@@
 F 0 "R3" H 2520 1496 50  0000 L CNN
 F 1 "100k" H 2520 1405 50  0000 L CNN
-F 2 "Resistor_THT:R_Axial_Default" V 2380 1450 50  0001 C CNN
+F 2 "Resistor_THT:R_Axial_DIN0204_L3.6mm_D1.6mm_P5.08mm_Horizontal" V 2380 1450 50  0001 C CNN
 F 3 "~" H 2450 1450 50  0001 C CNN
 	1    2450 1450
@@
 F 0 "R9" V 3493 2650 50  0000 C CNN
 F 1 "100k" V 3584 2650 50  0000 C CNN
-F 2 "Resistor_THT:R_Axial_Default" V 3630 2650 50  0001 C CNN
+F 2 "Resistor_THT:R_Axial_DIN0204_L3.6mm_D1.6mm_P5.08mm_Horizontal" V 3630 2650 50  0001 C CNN
 F 3 "~" H 3700 2650 50  0001 C CNN
 	1    3700 2650
@@
 F 0 "R6" V 2693 2650 50  0000 C CNN
 F 1 "100k" V 2784 2650 50  0000 C CNN
-F 2 "Resistor_THT:R_Axial_Default" V 2830 2650 50  0001 C CNN
+F 2 "Resistor_THT:R_Axial_DIN0204_L3.6mm_D1.6mm_P5.08mm_Horizontal" V 2830 2650 50  0001 C CNN
 F 3 "~" H 2900 2650 50  0001 C CNN
 	1    2900 2650
@@
 F 0 "R12" V 4343 2500 50  0000 C CNN
 F 1 "33k" V 4434 2500 50  0000 C CNN
-F 2 "Resistor_THT:R_Axial_Default" V 4480 2500 50  0001 C CNN
+F 2 "Resistor_THT:R_Axial_DIN0204_L3.6mm_D1.6mm_P5.08mm_Horizontal" V 4480 2500 50  0001 C CNN
 F 3 "~" H 4550 2500 50  0001 C CNN
 	1    4550 2500
@@
 F 0 "R11" V 4343 1200 50  0000 C CNN
 F 1 "33k" V 4434 1200 50  0000 C CNN
-F 2 "Resistor_THT:R_Axial_Default" V 4480 1200 50  0001 C CNN
+F 2 "Resistor_THT:R_Axial_DIN0204_L3.6mm_D1.6mm_P5.08mm_Horizontal" V 4480 1200 50  0001 C CNN
 F 3 "~" H 4550 1200 50  0001 C CNN
 	1    4550 1200
@@
 F 0 "R4" V 2393 2650 50  0000 C CNN
 F 1 "10k" V 2484 2650 50  0000 C CNN
-F 2 "Resistor_THT:R_Axial_Default" V 2530 2650 50  0001 C CNN
+F 2 "Resistor_THT:R_Axial_DIN0204_L3.6mm_D1.6mm_P5.08mm_Horizontal" V 2530 2650 50  0001 C CNN
 F 3 "~" H 2600 2650 50  0001 C CNN
 	1    2600 2650
@@
 F 0 "R7" H 2880 3454 50  0000 R CNN
 F 1 "100k" H 2880 3545 50  0000 R CNN
-F 2 "Resistor_THT:R_Axial_Default" V 2880 3500 50  0001 C CNN
+F 2 "Resistor_THT:R_Axial_DIN0204_L3.6mm_D1.6mm_P5.08mm_Horizontal" V 2880 3500 50  0001 C CNN
 F 3 "~" H 2950 3500 50  0001 C CNN
 	1    2950 3500
@@
 F 0 "R13" V 4343 3350 50  0000 C CNN
 F 1 "33k" V 4434 3350 50  0000 C CNN
-F 2 "Resistor_THT:R_Axial_Default" V 4480 3350 50  0001 C CNN
+F 2 "Resistor_THT:R_Axial_DIN0204_L3.6mm_D1.6mm_P5.08mm_Horizontal" V 4480 3350 50  0001 C CNN
 F 3 "~" H 4550 3350 50  0001 C CNN
 	1    4550 3350
@@
 F 0 "R14" H 5380 1404 50  0000 R CNN
 F 1 "100k" H 5380 1495 50  0000 R CNN
-F 2 "Resistor_THT:R_Axial_Default" V 5380 1450 50  0001 C CNN
+F 2 "Resistor_THT:R_Axial_DIN0204_L3.6mm_D1.6mm_P5.08mm_Horizontal" V 5380 1450 50  0001 C CNN
 F 3 "~" H 5450 1450 50  0001 C CNN
 	1    5450 1450
@@
 F 0 "R15" H 5380 2504 50  0000 R CNN
 F 1 "100k" H 5380 2595 50  0000 R CNN
-F 2 "Resistor_THT:R_Axial_Default" V 5380 2550 50  0001 C CNN
+F 2 "Resistor_THT:R_Axial_DIN0204_L3.6mm_D1.6mm_P5.08mm_Horizontal" V 5380 2550 50  0001 C CNN
 F 3 "~" H 5450 2550 50  0001 C CNN
 	1    5450 2550
@@
 F 0 "R18" V 7057 2400 50  0000 C CNN
 F 1 "10k" V 6966 2400 50  0000 C CNN
-F 2 "Resistor_THT:R_Axial_Default" V 6780 2400 50  0001 C CNN
+F 2 "Resistor_THT:R_Axial_DIN0204_L3.6mm_D1.6mm_P5.08mm_Horizontal" V 6780 2400 50  0001 C CNN
 F 3 "~" H 6850 2400 50  0001 C CNN
 	1    6850 2400
@@
 F 0 "R17" V 7057 1300 50  0000 C CNN
 F 1 "47k" V 6966 1300 50  0000 C CNN
-F 2 "Resistor_THT:R_Axial_Default" V 6780 1300 50  0001 C CNN
+F 2 "Resistor_THT:R_Axial_DIN0204_L3.6mm_D1.6mm_P5.08mm_Horizontal" V 6780 1300 50  0001 C CNN
 F 3 "~" H 6850 1300 50  0001 C CNN
 	1    6850 1300
@@
 F 0 "R19" H 7370 2096 50  0000 L CNN
 F 1 "10k" H 7370 2005 50  0000 L CNN
-F 2 "Resistor_THT:R_Axial_Default" V 7230 2050 50  0001 C CNN
+F 2 "Resistor_THT:R_Axial_DIN0204_L3.6mm_D1.6mm_P5.08mm_Horizontal" V 7230 2050 50  0001 C CNN
 F 3 "~" H 7300 2050 50  0001 C CNN
 	1    7300 2050
@@
 F 0 "R20" V 7857 2200 50  0000 C CNN
 F 1 "47k" V 7766 2200 50  0000 C CNN
-F 2 "Resistor_THT:R_Axial_Default" V 7580 2200 50  0001 C CNN
+F 2 "Resistor_THT:R_Axial_DIN0204_L3.6mm_D1.6mm_P5.08mm_Horizontal" V 7580 2200 50  0001 C CNN
 F 3 "~" H 7650 2200 50  0001 C CNN
 	1    7650 2200
@@
 F 0 "R22" V 9007 1200 50  0000 C CNN
 F 1 "100k" V 8916 1200 50  0000 C CNN
-F 2 "Resistor_THT:R_Axial_Default" V 8730 1200 50  0001 C CNN
+F 2 "Resistor_THT:R_Axial_DIN0204_L3.6mm_D1.6mm_P5.08mm_Horizontal" V 8730 1200 50  0001 C CNN
 F 3 "~" H 8800 1200 50  0001 C CNN
 	1    8800 1200
@@
 F 0 "R21" H 8120 2496 50  0000 L CNN
 F 1 "100k" H 8120 2405 50  0000 L CNN
-F 2 "Resistor_THT:R_Axial_Default" V 7980 2450 50  0001 C CNN
+F 2 "Resistor_THT:R_Axial_DIN0204_L3.6mm_D1.6mm_P5.08mm_Horizontal" V 7980 2450 50  0001 C CNN
 F 3 "~" H 8050 2450 50  0001 C CNN
 	1    8050 2450
@@
 F 0 "R16" V 6457 3550 50  0000 C CNN
 F 1 "4.7k" V 6366 3550 50  0000 C CNN
-F 2 "Resistor_THT:R_Axial_Default" V 6180 3550 50  0001 C CNN
+F 2 "Resistor_THT:R_Axial_DIN0204_L3.6mm_D1.6mm_P5.08mm_Horizontal" V 6180 3550 50  0001 C CNN
 F 3 "~" H 6250 3550 50  0001 C CNN
 	1    6250 3550
@@
 F 0 "R1" V 2357 4050 50  0000 C CNN
 F 1 "33k" V 2266 4050 50  0000 C CNN
-F 2 "Resistor_THT:R_Axial_Default" V 2080 4050 50  0001 C CNN
+F 2 "Resistor_THT:R_Axial_DIN0204_L3.6mm_D1.6mm_P5.08mm_Horizontal" V 2080 4050 50  0001 C CNN
 F 3 "~" H 2150 4050 50  0001 C CNN
 	1    2150 4050
@@
 F 0 "R2" V 2407 4450 50  0000 C CNN
 F 1 "33k" V 2316 4450 50  0000 C CNN
-F 2 "Resistor_THT:R_Axial_Default" V 2130 4450 50  0001 C CNN
+F 2 "Resistor_THT:R_Axial_DIN0204_L3.6mm_D1.6mm_P5.08mm_Horizontal" V 2130 4450 50  0001 C CNN
 F 3 "~" H 2200 4450 50  0001 C CNN
 	1    2200 4450
@@
 F 0 "R8" V 3357 4800 50  0000 C CNN
 F 1 "10k" V 3266 4800 50  0000 C CNN
-F 2 "Resistor_THT:R_Axial_Default" V 3080 4800 50  0001 C CNN
+F 2 "Resistor_THT:R_Axial_DIN0204_L3.6mm_D1.6mm_P5.08mm_Horizontal" V 3080 4800 50  0001 C CNN
 F 3 "~" H 3150 4800 50  0001 C CNN
 	1    3150 4800
@@
 F 0 "R10" V 3957 4300 50  0000 C CNN
 F 1 "10k" V 3866 4300 50  0000 C CNN
-F 2 "Resistor_THT:R_Axial_Default" V 3680 4300 50  0001 C CNN
+F 2 "Resistor_THT:R_Axial_DIN0204_L3.6mm_D1.6mm_P5.08mm_Horizontal" V 3680 4300 50  0001 C CNN
 F 3 "~" H 3750 4300 50  0001 C CNN
 	1    3750 4300
@@
 F 0 "R5" H 2680 5054 50  0000 R CNN
 F 1 "33k" H 2680 5145 50  0000 R CNN
-F 2 "Resistor_THT:R_Axial_Default" V 2680 5100 50  0001 C CNN
+F 2 "Resistor_THT:R_Axial_DIN0204_L3.6mm_D1.6mm_P5.08mm_Horizontal" V 2680 5100 50  0001 C CNN
 F 3 "~" H 2750 5100 50  0001 C CNN
 	1    2750 5100
